Commit message: mbx no prefix

File: urdf/mbx_arm_model.urdf.xacro (robot description, xacro)
@@ -1,5 +1,5 @@
 <?xml version="1.0"?>
 <robot name="robot" xmlns:xacro="http://www.ros.org/wiki/xacro">
-    <xacro:property name="ns" value="/mbx/" />
+    <xacro:property name="ns" value="" />
     <!-- variable -->
     <xacro:property name="PI" value="3.1415926"/>
@@ -489,6 +489,6 @@
     <gazebo>
         <plugin name="gazebo_ros_control" filename="libgazebo_ros_control.so">
-            <robotNamespace>/mbx</robotNamespace>
-            <robotParam>/mbx/robot_description</robotParam>
+            <robotNamespace>/</robotNamespace>
+            <robotParam>robot_description</robotParam>
             <robotSimType>gazebo_ros_control/DefaultRobotHWSim</robotSimType>
         </plugin>

File: urdf/ur10_robot.urdf.xacro (robot description, xacro)
@@ -8,5 +8,5 @@
   <xacro:include filename="$(find gazebo_example)/urdf/ur10.urdf.xacro" />
   <!-- arm -->
-  <xacro:ur10_robot prefix="/mbx/" joint_limited="false"
+  <xacro:ur10_robot prefix="" joint_limited="false"
     transmission_hw_interface="$(arg transmission_hw_interface)"
   />
