Commit message: add rviz config

File: urdf/iiwa_agv.urdf.xacro (robot description, xacro)
@@ -59,8 +59,4 @@
     <child
       link="${prefix}base_link" />
-    <axis
-      xyz="0 0 0" />
-    <safety_controller
-      k_velocity="0" />
   </joint>
     <!-- link list -->
@@ -492,8 +488,8 @@
     <plugin name="base_controller" filename="libgazebo_ros_planar_move.so">
       <commandTopic>cmd_vel</commandTopic>
-      <odometryTopic>odom</odometryTopic>
-      <odometryFrame>odom</odometryFrame>
+      <odometryTopic>world</odometryTopic>
+      <odometryFrame>world</odometryFrame>
       <odometryRate>20.0</odometryRate>
-      <robotBaseFrame>base_link</robotBaseFrame>
+      <robotBaseFrame>agv_link</robotBaseFrame>
     </plugin>
   </gazebo>

Commit message: rid of kuka pkg

File: urdf/iiwa_agv.urdf.xacro (robot description, xacro)
@@ -25,5 +25,5 @@
       <geometry>
         <mesh
-          filename="package://kuka_lbr_iiwa_support/meshes/che.STL" />
+          filename="package://gazebo_example/meshes/che.STL" />
       </geometry>
       <material
@@ -39,5 +39,5 @@
       <geometry>
         <mesh
-          filename="package://kuka_lbr_iiwa_support/meshes/che.STL" />
+          filename="package://gazebo_example/meshes/che.STL" />
       </geometry>
     </collision>
@@ -65,11 +65,11 @@
         <origin xyz="0 0 0" rpy="0 0 0" />
         <geometry>
-          <mesh filename="package://kuka_lbr_iiwa_support/meshes/lbr_iiwa_14_r820/visual/base_link.dae" />
-        </geometry>
-      </visual>
-      <collision>
-        <origin xyz="0 0 0" rpy="0 0 0" />
-        <geometry>
-          <mesh filename="package://kuka_lbr_iiwa_support/meshes/lbr_iiwa_14_r820/collision/base_link.stl" />
+          <mesh filename="package://gazebo_example/meshes/lbr_iiwa_14_r820/visual/base_link.dae" />
+        </geometry>
+      </visual>
+      <collision>
+        <origin xyz="0 0 0" rpy="0 0 0" />
+        <geometry>
+          <mesh filename="package://gazebo_example/meshes/lbr_iiwa_14_r820/collision/base_link.stl" />
         </geometry>
       </collision>
@@ -82,11 +82,11 @@
         <origin xyz="0 0 0" rpy="0 0 0" />
         <geometry>
-          <mesh filename="package://kuka_lbr_iiwa_support/meshes/lbr_iiwa_14_r820/visual/link_1.dae" />
-        </geometry>
-      </visual>
-      <collision>
-        <origin xyz="0 0 0" rpy="0 0 0" />
-        <geometry>
-          <mesh filename="package://kuka_lbr_iiwa_support/meshes/lbr_iiwa_14_r820/collision/link_1.stl" />
+          <mesh filename="package://gazebo_example/meshes/lbr_iiwa_14_r820/visual/link_1.dae" />
+        </geometry>
+      </visual>
+      <collision>
+        <origin xyz="0 0 0" rpy="0 0 0" />
+        <geometry>
+          <mesh filename="package://gazebo_example/meshes/lbr_iiwa_14_r820/collision/link_1.stl" />
         </geometry>
       </collision>
@@ -99,11 +99,11 @@
         <origin xyz="0 0 0" rpy="0 0 0" />
         <geometry>
-          <mesh filename="package://kuka_lbr_iiwa_support/meshes/lbr_iiwa_14_r820/visual/link_2.dae" />
-        </geometry>
-      </visual>
-      <collision>
-        <origin xyz="0 0 0" rpy="0 0 0" />
-        <geometry>
-          <mesh filename="package://kuka_lbr_iiwa_support/meshes/lbr_iiwa_14_r820/collision/link_2.stl" />
+          <mesh filename="package://gazebo_example/meshes/lbr_iiwa_14_r820/visual/link_2.dae" />
+        </geometry>
+      </visual>
+      <collision>
+        <origin xyz="0 0 0" rpy="0 0 0" />
+        <geometry>
+          <mesh filename="package://gazebo_example/meshes/lbr_iiwa_14_r820/collision/link_2.stl" />
         </geometry>
       </collision>
@@ -116,11 +116,11 @@
         <origin xyz="0 0 0" rpy="0 0 0" />
         <geometry>
-          <mesh filename="package://kuka_lbr_iiwa_support/meshes/lbr_iiwa_14_r820/visual/link_3.dae" />
-        </geometry>
-      </visual>
-      <collision>
-        <origin xyz="0 0 0" rpy="0 0 0" />
-        <geometry>
-          <mesh filename="package://kuka_lbr_iiwa_support/meshes/lbr_iiwa_14_r820/collision/link_3.stl" />
+          <mesh filename="package://gazebo_example/meshes/lbr_iiwa_14_r820/visual/link_3.dae" />
+        </geometry>
+      </visual>
+      <collision>
+        <origin xyz="0 0 0" rpy="0 0 0" />
+        <geometry>
+          <mesh filename="package://gazebo_example/meshes/lbr_iiwa_14_r820/collision/link_3.stl" />
         </geometry>
       </collision>
@@ -133,11 +133,11 @@
         <origin xyz="0 0 0" rpy="0 0 0" />
         <geometry>
-          <mesh filename="package://kuka_lbr_iiwa_support/meshes/lbr_iiwa_14_r820/visual/link_4.dae" />
-        </geometry>
-      </visual>
-      <collision>
-        <origin xyz="0 0 0" rpy="0 0 0" />
-        <geometry>
-          <mesh filename="package://kuka_lbr_iiwa_support/meshes/lbr_iiwa_14_r820/collision/link_4.stl" />
+          <mesh filename="package://gazebo_example/meshes/lbr_iiwa_14_r820/visual/link_4.dae" />
+        </geometry>
+      </visual>
+      <collision>
+        <origin xyz="0 0 0" rpy="0 0 0" />
+        <geometry>
+          <mesh filename="package://gazebo_example/meshes/lbr_iiwa_14_r820/collision/link_4.stl" />
         </geometry>
       </collision>
@@ -150,11 +150,11 @@
         <origin xyz="0 0 0" rpy="0 0 0" />
         <geometry>
-          <mesh filename="package://kuka_lbr_iiwa_support/meshes/lbr_iiwa_14_r820/visual/link_5.dae" />
-        </geometry>
-      </visual>
-      <collision>
-        <origin xyz="0 0 0" rpy="0 0 0" />
-        <geometry>
-          <mesh filename="package://kuka_lbr_iiwa_support/meshes/lbr_iiwa_14_r820/collision/link_5.stl" />
+          <mesh filename="package://gazebo_example/meshes/lbr_iiwa_14_r820/visual/link_5.dae" />
+        </geometry>
+      </visual>
+      <collision>
+        <origin xyz="0 0 0" rpy="0 0 0" />
+        <geometry>
+          <mesh filename="package://gazebo_example/meshes/lbr_iiwa_14_r820/collision/link_5.stl" />
         </geometry>
       </collision>
@@ -167,11 +167,11 @@
         <origin xyz="0 0 0" rpy="0 0 0" />
         <geometry>
-          <mesh filename="package://kuka_lbr_iiwa_support/meshes/lbr_iiwa_14_r820/visual/link_6.dae" />
-        </geometry>
-      </visual>
-      <collision>
-        <origin xyz="0 0 0" rpy="0 0 0" />
-        <geometry>
-          <mesh filename="package://kuka_lbr_iiwa_support/meshes/lbr_iiwa_14_r820/collision/link_6.stl" />
+          <mesh filename="package://gazebo_example/meshes/lbr_iiwa_14_r820/visual/link_6.dae" />
+        </geometry>
+      </visual>
+      <collision>
+        <origin xyz="0 0 0" rpy="0 0 0" />
+        <geometry>
+          <mesh filename="package://gazebo_example/meshes/lbr_iiwa_14_r820/collision/link_6.stl" />
         </geometry>
       </collision>
@@ -184,11 +184,11 @@
         <origin xyz="0 0 0" rpy="0 0 0" />
         <geometry>
-          <mesh filename="package://kuka_lbr_iiwa_support/meshes/lbr_iiwa_14_r820/visual/link_7.dae" />
-        </geometry>
-      </visual>
-      <collision>
-        <origin xyz="0 0 0" rpy="0 0 0" />
-        <geometry>
-          <mesh filename="package://kuka_lbr_iiwa_support/meshes/lbr_iiwa_14_r820/collision/link_7.stl" />
+          <mesh filename="package://gazebo_example/meshes/lbr_iiwa_14_r820/visual/link_7.dae" />
+        </geometry>
+      </visual>
+      <collision>
+        <origin xyz="0 0 0" rpy="0 0 0" />
+        <geometry>
+          <mesh filename="package://gazebo_example/meshes/lbr_iiwa_14_r820/collision/link_7.stl" />
         </geometry>
       </collision>
@@ -266,5 +266,5 @@
       <visual>
         <geometry>
-          <mesh filename="package://kuka_lbr_iiwa_support/meshes/pan.STL"/>
+          <mesh filename="package://gazebo_example/meshes/pan.STL"/>
         </geometry>
         <material name="black">
@@ -274,5 +274,5 @@
       <collision>
         <geometry>
-          <mesh filename="package://kuka_lbr_iiwa_support/meshes/pan.STL"/>
+          <mesh filename="package://gazebo_example/meshes/pan.STL"/>
         </geometry>
       </collision>
@@ -291,5 +291,5 @@
       <visual>
         <geometry>
-          <mesh filename="package://kuka_lbr_iiwa_support/meshes/xiao_arm.STL"/>
+          <mesh filename="package://gazebo_example/meshes/xiao_arm.STL"/>
         </geometry>
         <material name="black1">
@@ -299,5 +299,5 @@
       <collision>
         <geometry>
-          <mesh filename="package://kuka_lbr_iiwa_support/meshes/xiao_arm.STL"/>
+          <mesh filename="package://gazebo_example/meshes/xiao_arm.STL"/>
         </geometry>
       </collision>
@@ -316,5 +316,5 @@
       <visual>
         <geometry>
-          <mesh filename="package://kuka_lbr_iiwa_support/meshes/xiao_arm.STL"/>
+          <mesh filename="package://gazebo_example/meshes/xiao_arm.STL"/>
         </geometry>
         <material name="white1">
@@ -324,5 +324,5 @@
       <collision>
         <geometry>
-          <mesh filename="package://kuka_lbr_iiwa_support/meshes/xiao_arm.STL"/>
+          <mesh filename="package://gazebo_example/meshes/xiao_arm.STL"/>
         </geometry>
       </collision>
@@ -341,5 +341,5 @@
       <visual>
         <geometry>
-          <mesh filename="package://kuka_lbr_iiwa_support/meshes/xiangji.STL"/>
+          <mesh filename="package://gazebo_example/meshes/xiangji.STL"/>
         </geometry>
         <material name="white2">
@@ -349,5 +349,5 @@
       <collision>
         <geometry>
-          <mesh filename="package://kuka_lbr_iiwa_support/meshes/xiao_arm.STL"/>
+          <mesh filename="package://gazebo_example/meshes/xiao_arm.STL"/>
         </geometry>
       </collision>
